Commit message: xacro changes

File: sumitomo_ws/src/drivetrain/urdf/parts.xacro (robot description, xacro)
@@ -30,3 +30,4 @@
     </transmission>
 </xacro:macro>
+<!-- = Caster wheel = -->
 </robot>

File: sumitomo_ws/src/drivetrain/urdf/simple_agv.urdf (robot description, URDF)
Before this commit: robot simple_agv, 3 links, 2 joints
Links:
- removed link link0
- added link chassis; visual box size=0.65 0.5 0.3
- added link world_link
Joints:
- added joint world_link_to_chassis: type fixed, parent world_link, child chassis
- joint joint1: parent link0 -> chassis
- joint joint2: parent link0 -> chassis
