Commit message: working urdf of differential robot

File: sumitomo_ws/src/drivetrain/urdf/constants.xacro (robot description, xacro)
@@ -8,4 +8,6 @@
 <xacro:property name="wheel_base" value="0.10"/>
 <xacro:property name="wheel_radio" value="${base_height/2}"/>
+<!-- TODO: Correct the caster_rad value -->
+<xacro:property name="caster_rad" value="${wheel_radio}"/>
 <xacro:property name="trans_ratio" value="1"/>
 <!--Note: The direction should be signaled with as (1 || -1) -->

File: sumitomo_ws/src/drivetrain/urdf/parts.xacro (robot description, xacro)
@@ -1,33 +1,74 @@
 <?xml version="1.0"?>
 <robot xmlns:xacro="http://www.ros.org/wiki/xacro" name="simple_agv">
-<!-- Include constants xacro -->
-<xacro:include filename="$(find drivetrain)/urdf/constants.xacro" />
-<!-- === PARTS ONLY === -->
-<!-- = Wheels = -->
-<<xacro:macro name="wheel" params="direction">
-    <visual>
+  <!-- Include constants xacro -->
+  <xacro:include filename="$(find drivetrain)/urdf/constants.xacro" />
+  <!-- === PARTS ONLY === -->
+  <!-- = Wheels = -->
+  <xacro:macro name="wheel_block" params="side invert parent_link">
+    <!-- Link (physical part)-->
+    <link name="wheel_${side}">
+      <visual>
+        <!-- Shape -->
         <geometry>
-            <cylinder length="${wheel_base}" radius="${wheel_radio}"/>
+          <cylinder length="${wheel_base}" radius="${wheel_radio}"/>
         </geometry>
-        <origin rpy="${pi/2} 0 0" xyz="0 ${base_width/2} ${wheel_radio}"/>
+        <!-- Origin relative to the link's joint -->
+        <origin xyz= "0 0 0" rpy="${pi/2} 0 0"/>
         <material name="black">
-            <color rgba="0 0 0 1"/>
+          <color rgba="0 0 0 1"/>
         </material>
-    </visual>
-</xacro:macro>
-<!-- = Transmission = -->
-                                            <!--Note: I use "*" as a separator -->
-<xacro:macro name="transmission_block" params="*joint_name *count *direction">
-    <transmission name="trans_$(count)">
+      </visual>
+    </link>
+    <!-- Joint (connection between links) -->
+    <joint name="joint_wheel_${side}" type="continuous">
+      <parent link="${parent_link}"/>
+      <child link="wheel_${side}"/>
+      <origin xyz="0 ${(base_length/2)*invert} ${wheel_radio}"/>
+      <!-- Axis rotation-->
+      <axis xyz="0 1 0"/> <!-- rpy="0 0 0 -->
+      <!-- Joint limits (Newtons) (rad/s)-->
+      <limit effort="50" velocity="20"/>
+    </joint>
+    <!-- Transmission -->
+    <transmission name="trans_${side}">
+      <!-- Type -->
       <type>transmission_interface/SimpleTransmission</type>
-      <joint name="${joint_name}">
-        <hardwareInterface>PositionJointInterface</hardwareInterface>
+      <!-- Joint -->
+      <joint name="joint_wheel_${side}">
+        <hardwareInterface> hardware_interface/EffortJointInterface </hardwareInterface>
       </joint>
-      <actuator name="motor_{count}">
-        <hardwareInterface>PositionJointInterface</hardwareInterface>
+      <!-- Actuator -->
+      <actuator name="motor_{side}">
+        <hardwareInterface>hardware_interface/EffortJointInterface</hardwareInterface>
         <mechanicalReduction>1</mechanicalReduction>
       </actuator>
     </transmission>
-</xacro:macro>
-<!-- = Caster wheel = -->
+  </xacro:macro>
+  <!-- = Transmission = -->
+  <!--Note: I use "*" as a separator -->
+  <!-- <xacro:macro name="transmission_block" params="joint_name *side *direction">
+  </xacro:macro> -->
+  <!-- = Caster wheel = -->
+  <xacro:macro name="caster_wheel_block" params="dir_x *dir_y ">
+  <collision>
+    <origin xyz="{$base_length/2*dir_x} ${$base_length/2*dir_y} ${caster_rad}" rpy="0 0 0"/>
+    <geometry>
+      <sphere radius="${caster_rad}"/>
+    </geometry>
+    <surface>
+      <friction>
+        <ode>
+          <slip1>0.0</slip1>
+          <slip2>0.0</slip2>
+        </ode>
+      </friction>
+    </surface>
+  </collision>
+  <visual>
+    <origin xyz="{$base_length/2*dir_x} ${$base_length/2*dir_y} ${caster_rad}" rpy="0 0 0"/>
+    <geometry>
+      <sphere radius="${caster_rad}"/>
+    </geometry>
+  </visual>
+ </xacro:macro>
 </robot>

Commit message: neccesary changes to spawn with no error. TODO: place the robot in a new namespace

File: sumitomo_ws/src/drivetrain/urdf/constants.xacro (robot description, xacro)
@@ -8,4 +8,5 @@
 <xacro:property name="wheel_base" value="0.10"/>
 <xacro:property name="wheel_radio" value="${base_height/2}"/>
+<xacro:property name="wheel_mass" value="3"/>
 <!-- TODO: Correct the caster_rad value -->
 <xacro:property name="caster_rad" value="${wheel_radio}"/>

File: sumitomo_ws/src/drivetrain/urdf/parts.xacro (robot description, xacro)
@@ -4,4 +4,10 @@
   <xacro:include filename="$(find drivetrain)/urdf/constants.xacro" />
   <!-- === PARTS ONLY === -->
+  <!-- Wheel Inertia -->
+  <xacro:macro name="wheel_inertia" params="r l m">
+        <inertia  ixx="${m*(3*r*r+l*l)/12}" ixy = "0" ixz = "0"
+              iyy="${m*(3*r*r+l*l)/12}" iyz = "0"
+              izz="${m*r*r/2}" />
+  </xacro:macro>
   <!-- = Wheels = -->
   <xacro:macro name="wheel_block" params="side invert parent_link">
@@ -19,4 +25,18 @@
         </material>
       </visual>
+      <!-- Collission -->
+      <collision>
+        <origin xyz="0 0 0 " rpy="${(pi/2)*invert} 0 0"/>
+          <geometry>
+              <cylinder length="${wheel_base}" radius="${wheel_radio}"/>
+          </geometry>
+      </collision>
+      <!-- Inertial: Requred for Gazebo -->
+      <inertial>
+        <mass value="${wheel_mass}"/>
+        <!-- <origin xyz="0 0 0" rpy="${pi/2} 0 0"/> -->
+        <xacro:wheel_inertia r="${wheel_radio}" l="${wheel_base}" m="${wheel_mass}"/>
+      </inertial>
+      <!-- <joint_properties damping="0.0" friction="0.0"/> -->
     </link>
     <!-- Joint (connection between links) -->
@@ -40,5 +60,5 @@
       <!-- Actuator -->
       <actuator name="motor_${side}">
-        <hardwareInterface>hardware_interface/EffortJointInterface</hardwareInterface>
+        <hardwareInterface> hardware_interface/EffortJointInterface </hardwareInterface>
         <mechanicalReduction>1</mechanicalReduction>
       </actuator>

File: sumitomo_ws/src/drivetrain/urdf/simple_agv.xacro (robot description, xacro)
@@ -27,4 +27,16 @@
             </material>
         </visual>
+         <!-- Collission -->
+        <collision>
+            <origin xyz="0 0 0.3"/>
+            <geometry>
+                <box size="0.65 0.5 0.3"/>
+            </geometry>
+        </collision>
+        <!-- Inertial: Requred for Gazebo -->
+        <inertial>
+            <mass value="${wheel_mass}"/>
+            <inertia ixx="0.1" ixy="0.0" ixz="0.0" iyy="0.1" iyz="0.0" izz="0.1"/>
+        </inertial>
     </link>
     <!-- === Joint definition === -->
@@ -41,6 +53,9 @@
     <gazebo>
         <plugin name="gazebo_ros_control" filename="libgazebo_ros_control.so">
-            <robotNamespace>/drivetrain</robotNamespace>
+            <robotNamespace>/</robotNamespace>
         </plugin>
     </gazebo>
+    <gazebo reference="chassis">
+        <material>Gazebo/Orange</material>
+    </gazebo>
   </robot>

Commit message: urdf changes

File: sumitomo_ws/src/drivetrain/urdf/constants.xacro (robot description, xacro)
@@ -9,4 +9,7 @@
 <xacro:property name="wheel_radio" value="${base_height/2}"/>
 <xacro:property name="wheel_mass" value="3"/>
+<!-- === Mesh properties===-->
+<xacro:property name="mesh_scale" value="1.0 1.0 1.0"/>
+<xacro:property name="chassis_path" value="package://drivetrain/urdf/chasis.STL"/>
 <!-- TODO: Correct the caster_rad value -->
 <xacro:property name="caster_rad" value="${wheel_radio}"/>

File: sumitomo_ws/src/drivetrain/urdf/robot_innert.urdf (robot description, URDF)
Before this commit: robot simple_agv, 4 links, 3 joints
Links:
- link chassis: mass None -> 3; geometry collision mesh filename=package://drivetrain/urdf/chasis.STL scale=1.0 1.0 1.0; visual mesh filename=package://drivetrain/urdf/chasis.STL scale=1.0 1.0 1.0

File: sumitomo_ws/src/drivetrain/urdf/simple_agv.xacro (robot description, xacro)
@@ -20,5 +20,5 @@
         <visual>
             <geometry>
-                <box size="0.65 0.5 0.3"/>
+                <mesh filename="${chassis_path}" scale="${mesh_scale}"/>
             </geometry>
             <origin xyz="0 0 0.3"/>
@@ -31,5 +31,5 @@
             <origin xyz="0 0 0.3"/>
             <geometry>
-                <box size="0.65 0.5 0.3"/>
+                <mesh filename="${chassis_path}" scale="${mesh_scale}"/>
             </geometry>
         </collision>
@@ -59,3 +59,39 @@
         <material>Gazebo/Orange</material>
     </gazebo>
+    <gazebo>
+    <plugin name="differential_drive_controller" filename="libgazebo_ros_diff_drive.so">
+    <!-- Plugin update rate in Hz -->
+    <updateRate>50</updateRate>
+    <!-- Name of left joint, defaults to `left_joint` -->
+    <leftJoint>joint_wheel_left</leftJoint>
+    <!-- Name of right joint, defaults to `right_joint` -->
+    <rightJoint>joint_wheel_right</rightJoint>
+    <!-- The distance from the center of one wheel to the other, in meters, defaults to 0.34 m -->
+    <wheelSeparation>0.5380</wheelSeparation>
+    <!-- Diameter of the wheels, in meters, defaults to 0.15 m -->
+    <wheelDiameter>0.2410</wheelDiameter>
+    <!-- Wheel acceleration, in rad/s^2, defaults to 0.0 rad/s^2 -->
+    <wheelAcceleration>1.0</wheelAcceleration>
+    <!-- Maximum torque which the wheels can produce, in Nm, defaults to 5 Nm -->
+    <wheelTorque>20</wheelTorque>
+    <!-- Topic to receive geometry_msgs/Twist message commands, defaults to `cmd_vel` -->
+    <commandTopic>cmd_vel</commandTopic>
+    <!-- Topic to publish nav_msgs/Odometry messages, defaults to `odom` -->
+    <odometryTopic>odom</odometryTopic>
+    <!-- Odometry frame, defaults to `odom` -->
+    <odometryFrame>odom</odometryFrame>
+    <!-- Robot frame to calculate odometry from, defaults to `base_footprint` -->
+    <robotBaseFrame>chassis</robotBaseFrame>
+    <!-- Odometry source, 0 for ENCODER, 1 for WORLD, defaults to WORLD -->
+    <odometrySource>1</odometrySource>
+    <!-- Set to true to publish transforms for the wheel links, defaults to false -->
+    <publishWheelTF>true</publishWheelTF>
+    <!-- Set to true to publish transforms for the odometry, defaults to true -->
+    <publishOdom>true</publishOdom>
+    <!-- Set to true to publish sensor_msgs/JointState on /joint_states for the wheel joints, defaults to false -->
+    <publishWheelJointState>true</publishWheelJointState>
+    <!-- Set to true to swap right and left wheels, defaults to true -->
+    <legacyMode>false</legacyMode>
+  </plugin>
+  </gazebo>
   </robot>

Commit message: Lowered wheels to have a moving robot

File: sumitomo_ws/src/drivetrain/urdf/constants.xacro (robot description, xacro)
@@ -7,9 +7,11 @@
 <xacro:property name="base_length" value="0.65"/>
 <xacro:property name="wheel_base" value="0.10"/>
-<xacro:property name="wheel_radio" value="${base_height/2}"/>
-<xacro:property name="wheel_mass" value="3"/>
+<xacro:property name="wheel_radio" value="0.095"/>
+<xacro:property name="wheel_mass" value="1"/>
 <!-- === Mesh properties===-->
 <xacro:property name="mesh_scale" value="1.0 1.0 1.0"/>
-<xacro:property name="chassis_path" value="package://drivetrain/urdf/chasis.STL"/>
+<xacro:property name="chassis_path" value="package://drivetrain/urdf/base_link.STL"/>
+<xacro:property name="wheel_dist" value="0.57"/>
+<xacro:property name="chassis_weight" value="20"/>
 <!-- TODO: Correct the caster_rad value -->
 <xacro:property name="caster_rad" value="${wheel_radio}"/>

File: sumitomo_ws/src/drivetrain/urdf/parts.xacro (robot description, xacro)
@@ -20,5 +20,5 @@
         </geometry>
         <!-- Origin relative to the link's joint -->
-        <origin xyz= "0 0 0" rpy="${pi/2} 0 0"/>
+        <origin xyz= "0 0 0" rpy="${(pi/2)*invert} 0 0"/>
         <material name="black">
           <color rgba="0 0 0 0.5"/>
@@ -35,5 +35,5 @@
       <inertial>
         <mass value="${wheel_mass}"/>
-        <!-- <origin xyz="0 0 0" rpy="${pi/2} 0 0"/> -->
+        <!-- <origin xyz="0 0 0" rpy="${(pi/2)*invert} 0 0"/> -->
         <xacro:wheel_inertia r="${wheel_radio}" l="${wheel_base}" m="${wheel_mass}"/>
       </inertial>
@@ -44,9 +44,9 @@
       <parent link="${parent_link}"/>
       <child link="wheel_${side}"/>
-      <origin xyz="0 ${(base_length/2)*invert} ${wheel_radio}"/>
+      <origin xyz="0 ${(wheel_dist/2)*invert} ${wheel_radio - 0.002}"/>
       <!-- Axis rotation-->
-      <axis xyz="0 1 0"/> <!-- rpy="0 0 0 -->
+      <axis xyz="0 1 0" rpy="0 0 0"/> <!-- -->
       <!-- Joint limits (Newtons) (rad/s)-->
-      <limit effort="50" velocity="20"/>
+      <limit effort="5000" velocity="3000"/>
     </joint>
     <!-- Transmission -->

File: sumitomo_ws/src/drivetrain/urdf/robot.urdf (robot description, URDF)
Before this commit: robot simple_agv, 4 links, 3 joints
Links:
- link chassis: mass None -> 1; geometry collision mesh filename=package://drivetrain/urdf/base_link.STL scale=1.0 1.0 1.0; visual mesh filename=package://drivetrain/urdf/base_link.STL scale=1.0 1.0 1.0
- link wheel_left: mass None -> 1; geometry collision cylinder length=0.1 radius=0.085; visual cylinder length=0.1 radius=0.08
- link wheel_right: mass None -> 1; geometry collision cylinder length=0.1 radius=0.085; visual cylinder length=0.1 radius=0.085
Joints:
- joint joint_wheel_left: origin xyz=0 -0.325 0.15 -> xyz=0 -0.325 0.085
- joint joint_wheel_right: origin xyz=0 0.325 0.15 -> xyz=0 0.325 0.085

File: sumitomo_ws/src/drivetrain/urdf/simple_agv.xacro (robot description, xacro)
@@ -22,5 +22,5 @@
                 <mesh filename="${chassis_path}" scale="${mesh_scale}"/>
             </geometry>
-            <origin xyz="0 0 0.3"/>
+            <origin xyz="0 0 0" rpy="0 0 ${pi/2}"/>
             <material name="white">
                 <color rgba="0 0 1 1"/>
@@ -29,5 +29,5 @@
          <!-- Collission -->
         <collision>
-            <origin xyz="0 0 0.3"/>
+            <origin xyz="0 0 0" rpy="0 0 ${pi/2}"/>
             <geometry>
                 <mesh filename="${chassis_path}" scale="${mesh_scale}"/>
@@ -36,5 +36,5 @@
         <!-- Inertial: Requred for Gazebo -->
         <inertial>
-            <mass value="${wheel_mass}"/>
+            <mass value="${chassis_weight}"/>
             <inertia ixx="0.1" ixy="0.0" ixz="0.0" iyy="0.1" iyz="0.0" izz="0.1"/>
         </inertial>
@@ -68,25 +68,25 @@
     <rightJoint>joint_wheel_right</rightJoint>
     <!-- The distance from the center of one wheel to the other, in meters, defaults to 0.34 m -->
-    <wheelSeparation>0.5380</wheelSeparation>
+    <wheelSeparation>${wheel_dist}</wheelSeparation>
     <!-- Diameter of the wheels, in meters, defaults to 0.15 m -->
-    <wheelDiameter>0.2410</wheelDiameter>
+    <wheelDiameter>${wheel_radio*2}</wheelDiameter>
     <!-- Wheel acceleration, in rad/s^2, defaults to 0.0 rad/s^2 -->
-    <wheelAcceleration>1.0</wheelAcceleration>
+    <wheelAcceleration>100.0</wheelAcceleration>
     <!-- Maximum torque which the wheels can produce, in Nm, defaults to 5 Nm -->
-    <wheelTorque>20</wheelTorque>
+    <wheelTorque>500</wheelTorque>
     <!-- Topic to receive geometry_msgs/Twist message commands, defaults to `cmd_vel` -->
     <commandTopic>cmd_vel</commandTopic>
     <!-- Topic to publish nav_msgs/Odometry messages, defaults to `odom` -->
-    <odometryTopic>odom</odometryTopic>
+    <!-- <odometryTopic>odom</odometryTopic> -->
     <!-- Odometry frame, defaults to `odom` -->
-    <odometryFrame>odom</odometryFrame>
+    <!-- <odometryFrame>odom</odometryFrame> -->
     <!-- Robot frame to calculate odometry from, defaults to `base_footprint` -->
-    <robotBaseFrame>chassis</robotBaseFrame>
+    <!-- <robotBaseFrame>chassis</robotBaseFrame> -->
     <!-- Odometry source, 0 for ENCODER, 1 for WORLD, defaults to WORLD -->
-    <odometrySource>1</odometrySource>
+    <!-- <odometrySource>1</odometrySource> -->
     <!-- Set to true to publish transforms for the wheel links, defaults to false -->
     <publishWheelTF>true</publishWheelTF>
     <!-- Set to true to publish transforms for the odometry, defaults to true -->
-    <publishOdom>true</publishOdom>
+    <publishOdom>false</publishOdom>
     <!-- Set to true to publish sensor_msgs/JointState on /joint_states for the wheel joints, defaults to false -->
     <publishWheelJointState>true</publishWheelJointState>
