Commit message: before sumitomo

File: sumitomo_ws/src/drivetrain/urdf/simple_agv.xacro (robot description, xacro)
@@ -50,4 +50,52 @@
     <xacro:wheel_block side="right" invert = "1" parent_link = "chassis"/>
     <xacro:wheel_block side="left" invert = "-1" parent_link = "chassis"/>
+    <!--Camera-->
+    <joint name="camera_joint" type="fixed">
+        <parent link="chassis"/>
+        <child link="camera_link"/>
+        <origin xyz="0.305 0 0.08" rpy="0 0 0"/>
+    </joint>
+    <link name="camera_link">
+        <visual>
+            <geometry>
+                <box size="0.010 0.03 0.03"/>
+            </geometry>
+            <material name="red"/>
+        </visual>
+    </link>
+    <joint name="camera_optical_joint" type="fixed">
+        <parent link="camera_link"/>
+        <child link="camera_link_optical"/>
+        <origin xyz="0 0 0" rpy="${-pi/2} 0 ${-pi/2}"/>
+    </joint>
+    <link name="camera_link_optical"></link>
+    <gazebo reference="camera_link">
+        <material>Gazebo/Red</material>
+        <sensor name="camera" type="camera">
+            <pose> 0 0 0 0 0 0 </pose>
+            <visualize>true</visualize>
+            <update_rate>10</update_rate>
+            <camera>
+                <horizontal_fov>1.089</horizontal_fov>
+                <image>
+                    <format>R8G8B8</format>
+                    <width>640</width>
+                    <height>480</height>
+                </image>
+                <clip>
+                    <near>0.05</near>
+                    <far>8.0</far>
+                </clip>
+            </camera>
+            <plugin name="camera_controller" filename="libgazebo_ros_camera.so">
+    		<alwaysOn>true</alwaysOn>
+    		<updateRate>0.1</updateRate>
+    		<cameraName>camera</cameraName>
+    		<imageTopicName>image_raw</imageTopicName>
+    		<cameraInfoTopicName>camera_info</cameraInfoTopicName>
+                <frame_name>camera_link_optical</frame_name>
+            </plugin>
+        </sensor>
+    </gazebo>
     <!-- === Gazebo Plugin === -->
     <gazebo>
